File: customDevboard.kicad_pcb (KiCad board)
At the start: 2 copper layers, 39 x 39 mm, 83 parts, among them J1 USB_C_Receptacle_USB2.0_14P, J10 GPIO29_ADC3, J11 GND, J12 GPIO0, J13 GPIO1, J14 GPIO2, J15 GPIO3, J16 GPIO4, J17 GPIO5, J18 GPIO6, J19 GPIO7, J2 RUN, J20 GPIO8, J21 GPIO9, J22 Conn_01x01, J23 Conn_01x01, J24 Conn_01x01, J25 Conn_01x01, J26 Conn_01x01, J27 Conn_01x01, J28 Conn_01x01, J29 Conn_01x01, J3 3V3, J30 Conn_01x01, J31 Conn_01x01, J32 Conn_01x01, J33 Conn_01x01, J34 Conn_01x01, J35 Conn_01x01, J36 Conn_01x01, J37 Conn_01x01, J38 Conn_01x01, J39 Conn_01x01, J4 VBUS, J40 Conn_01x01, J41 Conn_01x01, J42 SWCLK, J43 GND, J44 SWD, J5 GND, J6 GND, J7 GPIO26_ADC0, J8 GPIO27_ADC1, J9 GPIO28_ADC2, SW1 BOOT, U1 RP2040, U2 W25Q128JVP, U3 TLV75733PDRV, Y1 12 MHz

Commit message: update pcb
Routing:
- net GND: track 46.4 -> 30.5 mm
Changed lines of the file:
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@@
-	)
-	(segment
-		(start 65.4875 64.6)
-		(end 66.1875 63.9)
-		(width 0.2)
-		(layer "B.Cu")
-		(net 1)
-	)
-	(segment
-		(start 47.5 65.5)
-		(end 47.5 71.75)
-		(width 0.2)
-		(layer "B.Cu")
-		(net 1)
-	)
-	(segment
-		(start 56.85 64.6)
-		(end 65.4875 64.6)
-		(width 0.2)
-		(layer "B.Cu")
-		(net 1)
 	)
 	(segment

Commit message: optimise
Routing:
- net GPIO25: track 52.6 -> 46.4 mm, vias 4 -> 2
- net +1V1: track 40.4 -> 39.9 mm, vias 5 -> 3
- net VBUS: vias 4 -> 2
Changed lines of the file:
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@@
+	)
+	(segment
+		(start 68 83)
+		(end 68 72.75)
+		(width 0.2)
+		(layer "F.Cu")
+		(net 2)
 	)
 	(segment
@@
 	)
 	(via
-		(at 68 83)
+		(at 68 72.75)
 		(size 0.6)
 		(drill 0.3)
@@
 	)
 	(segment
-		(start 68 83)
-		(end 68 55.75)
-		(width 0.2)
-		(layer "B.Cu")
-		(net 2)
-	)
-	(segment
 		(start 76.25 53.77)
 		(end 75.48 53)
@@
 	)
 	(segment
+		(start 68 55.75)
+		(end 70.75 53)
+		(width 0.2)
+		(layer "B.Cu")
+		(net 2)
+	)
+	(segment
 		(start 75.48 53)
 		(end 70.75 53)
@@
 	)
 	(segment
+		(start 68 72.75)
+		(end 68 55.75)
+		(width 0.2)
+		(layer "B.Cu")
+		(net 2)
+	)
+	(segment
 		(start 60.75 53)
 		(end 55.25 47.5)
-		(width 0.2)
-		(layer "B.Cu")
-		(net 2)
-	)
-	(segment
-		(start 68 55.75)
-		(end 70.75 53)
 		(width 0.2)
 		(layer "B.Cu")
@@
 		(end 78.25 61.23)
 		(width 0.5)
-		(layer "F.Cu")
-		(net 3)
-	)
-	(segment
-		(start 67.4 73.75)
-		(end 68.6 73.75)
-		(width 0.2)
 		(layer "F.Cu")
 		(net 3)
@@
 	)
 	(via
-		(at 67.4 73.75)
-		(size 0.6)
-		(drill 0.3)
-		(layers "F.Cu" "B.Cu")
-		(net 3)
-	)
-	(via
 		(at 71 66)
 		(size 0.6)
@@
 		(net 3)
 	)
-	(via
-		(at 68.6 73.75)
-		(size 0.6)
-		(drill 0.3)
-		(layers "F.Cu" "B.Cu")
-		(net 3)
-	)
 	(segment
 		(start 71 66)
@@
 	)
 	(segment
+		(start 63.711524 66.404797)
+		(end 67.25 69.943273)
+		(width 0.2)
+		(layer "B.Cu")
+		(net 3)
+	)
+	(segment
+		(start 67.25 73.6)
+		(end 67.4 73.75)
+		(width 0.2)
+		(layer "B.Cu")
+		(net 3)
+	)
+	(segment
+		(start 69.5 72.75)
+		(end 69.5 67.5)
+		(width 0.2)
+		(layer "B.Cu")
+		(net 3)
+	)
+	(segment
+		(start 67.4 73.75)
+		(end 68.5 73.75)
+		(width 0.2)
+		(layer "B.Cu")
+		(net 3)
+	)
+	(segment
+		(start 67.25 69.943273)
+		(end 67.25 73.6)
+		(width 0.2)
+		(layer "B.Cu")
+		(net 3)
+	)
+	(segment
+		(start 69.5 67.5)
+		(end 71 66)
+		(width 0.2)
+		(layer "B.Cu")
+		(net 3)
+	)
+	(segment
 		(start 68.5 73.75)
-		(end 68.401 73.651)
-		(width 0.2)
-		(layer "B.Cu")
-		(net 3)
-	)
-	(segment
-		(start 63.711524 66.404797)
-		(end 67.599 70.292273)
-		(width 0.2)
-		(layer "B.Cu")
-		(net 3)
-	)
-	(segment
-		(start 68.401 68.599)
-		(end 71 66)
-		(width 0.2)
-		(layer "B.Cu")
-		(net 3)
-	)
-	(segment
-		(start 67.599 70.292273)
-		(end 67.599 73.551)
-		(width 0.2)
-		(layer "B.Cu")
-		(net 3)
-	)
-	(segment
-		(start 68.401 73.651)
-		(end 68.401 68.599)
-		(width 0.2)
-		(layer "B.Cu")
-		(net 3)
-	)
-	(segment
-		(start 68.6 73.75)
-		(end 68.5 73.75)
-		(width 0.2)
-		(layer "B.Cu")
-		(net 3)
-	)
-	(segment
-		(start 67.599 73.551)
-		(end 67.4 73.75)
+		(end 69.5 72.75)
 		(width 0.2)
 		(layer "B.Cu")
@@
 		(start 78.068 68.786)
 		(end 78.482 69.2)
-		(width 0.2)
-		(layer "F.Cu")
-		(net 4)
-	)
-	(segment
-		(start 68.6 74.550003)
-		(end 67.4 74.550003)
 		(width 0.2)
 		(layer "F.Cu")
@@
 		(net 4)
 	)
-	(via
-		(at 68.6 74.550003)
-		(size 0.6)
-		(drill 0.3)
-		(layers "F.Cu" "B.Cu")
-		(net 4)
-	)
-	(via
-		(at 67.4 74.550003)
-		(size 0.6)
-		(drill 0.3)
-		(layers "F.Cu" "B.Cu")
+	(segment
+		(start 69.199997 74.550003)
+		(end 67.4 74.550003)
+		(width 0.2)
+		(layer "B.Cu")
+		(net 4)
+	)
+	(segment
+		(start 67.4 74.550003)
+		(end 59.550003 74.550003)
+		(width 0.2)
+		(layer "B.Cu")
+		(net 4)
+	)
+	(segment
+		(start 74.75 69)
+		(end 69.199997 74.550003)
+		(width 0.2)
+		(layer "B.Cu")
 		(net 4)
 	)
@@
 	)
 	(segment
-		(start 67.4 74.550003)
-		(end 59.550003 74.550003)
-		(width 0.2)
-		(layer "B.Cu")
-		(net 4)
-	)
-	(segment
-		(start 69.199997 74.550003)
-		(end 68.6 74.550003)
-		(width 0.2)
-		(layer "B.Cu")
-		(net 4)
-	)
-	(segment
-		(start 74.75 69)
-		(end 69.199997 74.550003)
-		(width 0.2)
-		(layer "B.Cu")
-		(net 4)
-	)
-	(segment
 		(start 59.550003 74.550003)
 		(end 47.5 62.5)
@@
 	)
 	(segment
-		(start 66.7875 67.3375)
+		(start 65 72)
 		(end 66.7875 70.2125)
 		(width 0.2)
@@
 	)
 	(segment
-		(start 67.4 75.350006)
-		(end 68.6 75.350006)
+		(start 65 75.5)
+		(end 65 72)
 		(width 0.2)
 		(layer "F.Cu")
@@
 	)
 	(segment
+		(start 65 83)
+		(end 65 75.5)
+		(width 0.2)
+		(layer "F.Cu")
+		(net 28)
+	)
+	(segment
 		(start 66.7875 70.2125)
-		(end 65 72)
-		(width 0.2)
-		(layer "F.Cu")
-		(net 28)
-	)
-	(segment
-		(start 65 72)
-		(end 65 83)
-		(width 0.2)
-		(layer "F.Cu")
-		(net 28)
-	)
-	(via
-		(at 67.4 75.350006)
-		(size 0.6)
-		(drill 0.3)
-		(layers "F.Cu" "B.Cu")
-		(net 28)
-	)
-	(via
-		(at 68.6 75.350006)
-		(size 0.6)
-		(drill 0.3)
-		(layers "F.Cu" "B.Cu")
+		(end 66.7875 67.3375)
+		(width 0.2)
+		(layer "F.Cu")
 		(net 28)
 	)
@@
 	)
 	(via
-		(at 65 83)
+		(at 65 75.5)
 		(size 0.6)
 		(drill 0.3)
@@
 	)
 	(segment
-		(start 65 77.750006)
+		(start 69.249937 75.350006)
+		(end 75.871 68.728943)
+		(width 0.2)
+		(layer "B.Cu")
+		(net 28)
+	)
+	(segment
+		(start 67.4 75.350006)
+		(end 69.249937 75.350006)
+		(width 0.2)
+		(layer "B.Cu")
+		(net 28)
+	)
+	(segment
+		(start 75.871 66.08)
+		(end 82.361 59.59)
+		(width 0.2)
+		(layer "B.Cu")
+		(net 28)
+	)
+	(segment
+		(start 67.250006 75.5)
 		(end 67.4 75.350006)
 		(width 0.2)
@@
 	)
 	(segment
+		(start 65 75.5)
+		(end 67.250006 75.5)
+		(width 0.2)
+		(layer "B.Cu")
+		(net 28)
+	)
+	(segment
 		(start 82.361 59.59)
-		(end 75.871 66.08)
+		(end 82.361 57.371)
+		(width 0.2)
+		(layer "B.Cu")
+		(net 28)
+	)
+	(segment
+		(start 82.361 57.371)
+		(end 80.74 55.75)
 		(width 0.2)
 		(layer "B.Cu")
@@
 		(width 0.2)
 		(layer "B.Cu")
-		(net 28)
-	)
-	(segment
-		(start 82.361 57.371)
-		(end 82.361 59.59)
-		(width 0.2)
-		(layer "B.Cu")
-		(net 28)
-	)
-	(segment
-		(start 69.249937 75.350006)
-		(end 75.871 68.728943)
-		(width 0.2)
-		(layer "B.Cu")
-		(net 28)
-	)
-	(segment
-		(start 65 83)
-		(end 65 77.750006)
-		(width 0.2)
-		(layer "B.Cu")
-		(net 28)
-	)
-	(segment
-		(start 68.6 75.350006)
-		(end 69.249937 75.350006)
-		(width 0.2)
-		(layer "B.Cu")
-		(net 28)
-	)
-	(segment
-		(start 80.74 55.75)
-		(end 82.361 57.371)
-		(width 0.2)
-		(layer "B.Cu")
