File: customDevboard.kicad_sch (KiCad schematic)
At the start: 78 parts, among them J1 USB_C_Receptacle_USB2.0_14P, J10 GPIO29_ADC3, J11 GND, J12 GPIO0, J13 GPIO1, J14 GPIO2, J15 GPIO3, J16 GPIO4, J17 GPIO5, J18 GPIO6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

Commit message: optimise
Other:
- moved on the sheet: C1, C10, C11, C12, C15, C16, C17, C2, C3, C4, C5, C6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
